File: eagle/taad.sch (EAGLE design)
At the start: 60 parts, among them IC1 LD117AS33TR, Q1 16 MHz, X1 MINI-USB-32005-201

Commit message: Routed everything
Parts:
- removed JP2: (no value), pinhead:PINHD-2X8
- added JP5, JP6: (no value), pinhead:PINHD-2X4
Connections:
- net +3V3: now also JP5.1, JP5.3, JP5.5, JP5.7; no longer JP2.1, JP2.3, JP2.5, JP2.7
- net +5V: now also JP6.1, JP6.3, JP6.5, JP6.7; no longer JP2.11, JP2.13, JP2.15, JP2.9
- net GND: now also JP5.2, JP5.4, JP5.6, JP5.8, JP6.2, JP6.4, JP6.6, JP6.8; no longer JP2.10, JP2.12, JP2.14, JP2.16, JP2.2, JP2.4, JP2.6, JP2.8
Changed lines of the file:
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@@
 <part name="GND15" library="supply1" deviceset="GND" device=""/>
 <part name="+3V6" library="supply1" deviceset="+3V3" device=""/>
-<part name="JP2" library="pinhead" deviceset="PINHD-2X8" device=""/>
 <part name="+3V8" library="supply1" deviceset="+3V3" device=""/>
 <part name="P+3" library="supply1" deviceset="+5V" device=""/>
@@
 <part name="GND18" library="supply1" deviceset="GND" device=""/>
 <part name="JP4" library="pinhead" deviceset="PINHD-1X1" device=""/>
+<part name="JP5" library="pinhead" deviceset="PINHD-2X4" device=""/>
+<part name="JP6" library="pinhead" deviceset="PINHD-2X4" device=""/>
 </parts>
 <sheets>
@@
 <instance part="GND15" gate="1" x="241.3" y="233.68"/>
 <instance part="+3V6" gate="G$1" x="261.62" y="233.68" rot="R180"/>
-<instance part="JP2" gate="A" x="-5.08" y="337.82" rot="R90"/>
 <instance part="+3V8" gate="G$1" x="-35.56" y="327.66" rot="R90"/>
-<instance part="P+3" gate="1" x="25.4" y="327.66" rot="R270"/>
+<instance part="P+3" gate="1" x="30.48" y="327.66" rot="R270"/>
 <instance part="GND19" gate="1" x="-38.1" y="350.52" rot="R270"/>
 <instance part="RN1" gate="A" x="162.56" y="314.96" rot="R90"/>
@@
 <instance part="GND18" gate="1" x="-88.9" y="96.52" rot="R90"/>
 <instance part="JP4" gate="G$1" x="-109.22" y="182.88" rot="R90"/>
+<instance part="JP5" gate="A" x="-7.62" y="337.82" rot="R90"/>
+<instance part="JP6" gate="A" x="7.62" y="337.82" rot="R90"/>
 </instances>
 <busses>
@@
 </segment>
 <segment>
-<pinref part="JP2" gate="A" pin="16"/>
 <wire x1="-35.56" y1="350.52" x2="-12.7" y2="350.52" width="0.1524" layer="91"/>
 <wire x1="-12.7" y1="350.52" x2="-10.16" y2="350.52" width="0.1524" layer="91"/>
 <wire x1="-10.16" y1="350.52" x2="-7.62" y2="350.52" width="0.1524" layer="91"/>
 <wire x1="-7.62" y1="350.52" x2="-5.08" y2="350.52" width="0.1524" layer="91"/>
-<wire x1="-5.08" y1="350.52" x2="-2.54" y2="350.52" width="0.1524" layer="91"/>
-<wire x1="-2.54" y1="350.52" x2="0" y2="350.52" width="0.1524" layer="91"/>
-<wire x1="0" y1="350.52" x2="2.54" y2="350.52" width="0.1524" layer="91"/>
+<wire x1="-5.08" y1="350.52" x2="2.54" y2="350.52" width="0.1524" layer="91"/>
 <wire x1="2.54" y1="350.52" x2="5.08" y2="350.52" width="0.1524" layer="91"/>
-<wire x1="5.08" y1="350.52" x2="5.08" y2="342.9" width="0.1524" layer="91"/>
-<pinref part="JP2" gate="A" pin="14"/>
+<wire x1="5.08" y1="350.52" x2="7.62" y2="350.52" width="0.1524" layer="91"/>
+<wire x1="7.62" y1="350.52" x2="10.16" y2="350.52" width="0.1524" layer="91"/>
+<wire x1="10.16" y1="350.52" x2="10.16" y2="342.9" width="0.1524" layer="91"/>
+<wire x1="7.62" y1="342.9" x2="7.62" y2="350.52" width="0.1524" layer="91"/>
+<wire x1="5.08" y1="342.9" x2="5.08" y2="350.52" width="0.1524" layer="91"/>
 <wire x1="2.54" y1="342.9" x2="2.54" y2="350.52" width="0.1524" layer="91"/>
-<pinref part="JP2" gate="A" pin="12"/>
-<wire x1="0" y1="342.9" x2="0" y2="350.52" width="0.1524" layer="91"/>
-<pinref part="JP2" gate="A" pin="10"/>
-<wire x1="-2.54" y1="342.9" x2="-2.54" y2="350.52" width="0.1524" layer="91"/>
-<pinref part="JP2" gate="A" pin="8"/>
 <wire x1="-5.08" y1="342.9" x2="-5.08" y2="350.52" width="0.1524" layer="91"/>
-<pinref part="JP2" gate="A" pin="6"/>
 <wire x1="-7.62" y1="342.9" x2="-7.62" y2="350.52" width="0.1524" layer="91"/>
-<pinref part="JP2" gate="A" pin="4"/>
 <wire x1="-10.16" y1="342.9" x2="-10.16" y2="350.52" width="0.1524" layer="91"/>
-<pinref part="JP2" gate="A" pin="2"/>
 <wire x1="-12.7" y1="342.9" x2="-12.7" y2="350.52" width="0.1524" layer="91"/>
 <pinref part="GND19" gate="1" pin="GND"/>
@@
 <junction x="-7.62" y="350.52"/>
 <junction x="-5.08" y="350.52"/>
-<junction x="-2.54" y="350.52"/>
-<junction x="0" y="350.52"/>
 <junction x="2.54" y="350.52"/>
 <junction x="5.08" y="350.52"/>
+<junction x="7.62" y="350.52"/>
+<junction x="10.16" y="350.52"/>
+<pinref part="JP5" gate="A" pin="2"/>
+<pinref part="JP5" gate="A" pin="4"/>
+<pinref part="JP5" gate="A" pin="6"/>
+<pinref part="JP5" gate="A" pin="8"/>
+<pinref part="JP6" gate="A" pin="2"/>
+<pinref part="JP6" gate="A" pin="4"/>
+<pinref part="JP6" gate="A" pin="6"/>
+<pinref part="JP6" gate="A" pin="8"/>
 </segment>
 <segment>
@@
 <segment>
 <pinref part="+3V8" gate="G$1" pin="+3V3"/>
-<pinref part="JP2" gate="A" pin="1"/>
 <wire x1="-33.02" y1="327.66" x2="-12.7" y2="327.66" width="0.1524" layer="91"/>
 <wire x1="-12.7" y1="327.66" x2="-12.7" y2="335.28" width="0.1524" layer="91"/>
-<pinref part="JP2" gate="A" pin="3"/>
 <wire x1="-12.7" y1="327.66" x2="-10.16" y2="327.66" width="0.1524" layer="91"/>
 <wire x1="-10.16" y1="327.66" x2="-10.16" y2="335.28" width="0.1524" layer="91"/>
-<pinref part="JP2" gate="A" pin="5"/>
 <wire x1="-10.16" y1="327.66" x2="-7.62" y2="327.66" width="0.1524" layer="91"/>
 <wire x1="-7.62" y1="327.66" x2="-7.62" y2="335.28" width="0.1524" layer="91"/>
-<pinref part="JP2" gate="A" pin="7"/>
 <wire x1="-7.62" y1="327.66" x2="-5.08" y2="327.66" width="0.1524" layer="91"/>
 <wire x1="-5.08" y1="327.66" x2="-5.08" y2="335.28" width="0.1524" layer="91"/>
@@
 <junction x="-12.7" y="327.66"/>
 <junction x="-7.62" y="327.66"/>
+<pinref part="JP5" gate="A" pin="1"/>
+<pinref part="JP5" gate="A" pin="3"/>
+<pinref part="JP5" gate="A" pin="5"/>
+<pinref part="JP5" gate="A" pin="7"/>
 </segment>
 <segment>
@@
 <segment>
 <pinref part="P+3" gate="1" pin="+5V"/>
-<pinref part="JP2" gate="A" pin="15"/>
-<wire x1="22.86" y1="327.66" x2="5.08" y2="327.66" width="0.1524" layer="91"/>
+<wire x1="27.94" y1="327.66" x2="10.16" y2="327.66" width="0.1524" layer="91"/>
+<wire x1="10.16" y1="327.66" x2="10.16" y2="335.28" width="0.1524" layer="91"/>
+<wire x1="10.16" y1="327.66" x2="7.62" y2="327.66" width="0.1524" layer="91"/>
+<wire x1="7.62" y1="327.66" x2="7.62" y2="335.28" width="0.1524" layer="91"/>
+<wire x1="7.62" y1="327.66" x2="5.08" y2="327.66" width="0.1524" layer="91"/>
 <wire x1="5.08" y1="327.66" x2="5.08" y2="335.28" width="0.1524" layer="91"/>
-<pinref part="JP2" gate="A" pin="13"/>
 <wire x1="5.08" y1="327.66" x2="2.54" y2="327.66" width="0.1524" layer="91"/>
 <wire x1="2.54" y1="327.66" x2="2.54" y2="335.28" width="0.1524" layer="91"/>
-<pinref part="JP2" gate="A" pin="11"/>
-<wire x1="2.54" y1="327.66" x2="0" y2="327.66" width="0.1524" layer="91"/>
-<wire x1="0" y1="327.66" x2="0" y2="335.28" width="0.1524" layer="91"/>
-<pinref part="JP2" gate="A" pin="9"/>
-<wire x1="0" y1="327.66" x2="-2.54" y2="327.66" width="0.1524" layer="91"/>
-<wire x1="-2.54" y1="327.66" x2="-2.54" y2="335.28" width="0.1524" layer="91"/>
-<junction x="0" y="327.66"/>
-<junction x="2.54" y="327.66"/>
 <junction x="5.08" y="327.66"/>
-</segment>
-</net>
+<junction x="7.62" y="327.66"/>
+<junction x="10.16" y="327.66"/>
+<pinref part="JP6" gate="A" pin="1"/>
+<pinref part="JP6" gate="A" pin="3"/>
+<pinref part="JP6" gate="A" pin="5"/>
+<pinref part="JP6" gate="A" pin="7"/>
+</segment>
+</net>

Commit message: Simplified form of PCB. Rerouted everything
Parts:
- removed CPUIN1, CPUIN2, CPUIN3, CPUIN4: 100n, rcl:C-EUC0805
- removed JP5, JP6: (no value), pinhead:PINHD-2X4
- added JP2: (no value), pinhead:PINHD-2X6
- renumbered ACC1 to C10, ACC2 to C11, ACC3 to C9, ACC4 to C8, CC1 to C13, CC2 to C12, CC3 to C14, CPUIN5 to C3, CPUOUT1 to C4, CPUOUT2 to C5, ESC1_CONN to JE1, ESC2_CONN to JE2, ESC3_CONN to JE3, LDOC1 to C2, LDOC2 to C1, LED_3V1 to L3, LED_3V2 to L2, LED_3V3 to L1, LED_5V to L4, PWMC to C15, R_3V1 to R6, R_3V2 to R7, R_3V3 to R1, R_5V to R10, SRV1_CONN to JS1, SRV2_CONN to JS2, SRV3_CONN to JS3, SRV4_CONN to JS4, SRV5_CONN to JS5, SRV6_CONN to JS6, TWI_CR to R8, TWI_DR to R9, USBD to 2, USBD1 to D1, USBR1 to R2, USBR2 to R3, USBR3 to R4, USBR4 to R5, XINC to C6, XOUTC to C7
Connections:
- net +3V3: now also JP2.1, JP2.3, JP2.5; no longer CPUIN1.2, CPUIN2.2, CPUIN3.2, CPUIN4.2, JP5.1, JP5.3, JP5.5, JP5.7
- net +5V: now also JP2.11, JP2.7, JP2.9; no longer JP6.1, JP6.3, JP6.5, JP6.7
- net GND: now also JP2.10, JP2.12, JP2.2, JP2.4, JP2.6, JP2.8; no longer CPUIN1.1, CPUIN2.1, CPUIN3.1, CPUIN4.1, JP5.2, JP5.4, JP5.6, JP5.8, JP6.2, JP6.4, JP6.6, JP6.8
- net SRV3: now also JS5.3; no longer JS3.3
- net SRV5: now also JS3.3; no longer JS5.3
