File: eagle/taad.brd (EAGLE design)
At the start: 85.8 x 74.3 mm, 56 parts, among them IC1 LD117AS33TR, Q1 16 MHz

Commit message: Changed 100nF to 0.1µF (same value different marking)
Parts:
- C1, C10, C2, C4, C9: value 100n -> 0.1µ
Changed lines of the file:
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@@
 <element name="R5" library="resistor" package="R0805" value="47k" x="23.622" y="40.64" rot="MR270"/>
 <element name="IC1" library="v-reg" package="SOT223" value="LD117AS33TR" x="41.402" y="70.104" rot="R270"/>
-<element name="C2" library="resistor" package="C0805" value="100n" x="31.242" y="67.31" rot="R180"/>
-<element name="C1" library="resistor" package="C0805" value="100n" x="47.752" y="70.104" rot="R90"/>
+<element name="C2" library="resistor" package="C0805" value="0.1µ" x="31.242" y="67.31" rot="R180"/>
+<element name="C1" library="resistor" package="C0805" value="0.1µ" x="47.752" y="70.104" rot="R90"/>
 <element name="L1" library="led" package="CHIP-LED0805" value="" x="31.242" y="65.278" rot="R270"/>
 <element name="R1" library="resistor" package="R0805" value="160" x="31.242" y="63.246" rot="R180"/>
@@
 </element>
 <element name="C11" library="rcl" package="C0805" value="10µ" x="38.862" y="34.29" rot="R90"/>
-<element name="C10" library="rcl" package="C0805" value="100n" x="38.354" y="38.354" rot="R90"/>
-<element name="C9" library="rcl" package="C0805" value="100n" x="47.752" y="32.766" rot="R270"/>
+<element name="C10" library="rcl" package="C0805" value="0.1µ" x="38.354" y="38.354" rot="R90"/>
+<element name="C9" library="rcl" package="C0805" value="0.1µ" x="47.752" y="32.766" rot="R270"/>
 <element name="I/O-PWM" library="max696x" package="QSOP16" value="" x="54.864" y="48.006" rot="MR180"/>
 <element name="2" library="diode" package="SOD123" value="" x="27.178" y="59.69" rot="MR270"/>
@@
 </element>
 <element name="C14" library="rcl" package="C0805" value="0.1µ" x="48.768" y="55.88" rot="R270"/>
-<element name="C4" library="rcl" package="C0805" value="100n" x="33.782" y="16.51" rot="MR0"/>
+<element name="C4" library="rcl" package="C0805" value="0.1µ" x="33.782" y="16.51" rot="MR0"/>
 <element name="D1" library="diode" package="SOD123" value="" x="27.178" y="66.04" rot="R90"/>
 <element name="JP3" library="pinhead" package="1X05" value="" x="42.926" y="4.064" rot="MR180"/>
